Commit message: feat(mola): allow for ground truth and estimated tf

File: stonefish_ws/src/MOLA_AUV/mola_auv_sim/urdf/materials.xacro (robot description, xacro)
@@ -16,4 +16,7 @@
         <color rgba="0.898 0.769 0.145 1.0"/>
     </material>
+    <material name="gray">
+        <color rgba="0.5 0.5 0.5 0.7"/>
+    </material>
     <material name="base">
         <texture filename="package://mola_auv_sim/data/mola_auv/texture/base.png"/>
